File: .kicad_proj/221.sch (KiCad schematic (older format))
At the start: 3 parts, among them U1 ATmega328-PU

Commit message: Add schematics 9, 10, 11 and 12
Changed lines of the file:
@@
 $Descr A4 11693 8268
 encoding utf-8
-Sheet 5 9
+Sheet 5 19
 Title ""
 Date ""
@@
 AR Path="/607BD0C6" Ref="U?"  Part="1"
 AR Path="/607B2C9D/607BD0C6" Ref="U1"  Part="1"
-F 0 "U1" H 4306 3546 50  0000 R CNN
+AR Path="/60A3FFA8/607BD0C6" Ref="U?"  Part="1"
+F 0 "U?" H 4306 3546 50  0000 R CNN
 F 1 "ATmega328-PU" H 4306 3455 50  0000 R CNN
 F 2 "Package_DIP:DIP-28_W7.62mm" H 4950 3500 50  0001 C CIN
@@
 AR Path="/607BD0CC" Ref="R?"  Part="1"
 AR Path="/607B2C9D/607BD0CC" Ref="R1"  Part="1"
-F 0 "R1" V 5943 2800 50  0000 C CNN
+AR Path="/60A3FFA8/607BD0CC" Ref="R?"  Part="1"
+F 0 "R?" V 5943 2800 50  0000 C CNN
 F 1 "60" V 6034 2800 50  0000 C CNN
 F 2 "" V 6080 2800 50  0001 C CNN
@@
 AR Path="/607BD0D3" Ref="D?"  Part="1"
 AR Path="/607B2C9D/607BD0D3" Ref="D1"  Part="1"
-F 0 "D1" H 6693 2545 50  0000 C CNN
+AR Path="/60A3FFA8/607BD0D3" Ref="D?"  Part="1"
+F 0 "D?" H 6693 2545 50  0000 C CNN
 F 1 "Blue LED" H 6693 2636 50  0000 C CNN
 F 2 "" H 6700 2800 50  0001 C CNN
@@
 AR Path="/607BD0DA" Ref="#PWR?"  Part="1"
 AR Path="/607B2C9D/607BD0DA" Ref="#PWR?"  Part="1"
+AR Path="/60A3FFA8/607BD0DA" Ref="#PWR?"  Part="1"
 F 0 "#PWR?" H 7000 2750 50  0001 C CNN
 F 1 "GND" H 7005 2827 50  0000 C CNN
@@
 $Comp
 L power:GND #PWR?
-U 1 1 607BD0E2
+U 1 1 60A41525
 P 4950 5000
-AR Path="/607BD0E2" Ref="#PWR?"  Part="1"
-AR Path="/607B2C9D/607BD0E2" Ref="#PWR?"  Part="1"
+AR Path="/60A41525" Ref="#PWR?"  Part="1"
+AR Path="/607B2C9D/60A41525" Ref="#PWR?"  Part="1"
+AR Path="/60A3FFA8/60A41525" Ref="#PWR?"  Part="1"
 F 0 "#PWR?" H 4950 4750 50  0001 C CNN
 F 1 "GND" H 4955 4827 50  0000 C CNN
@@
 $Comp
 L power:+5V #PWR?
-U 1 1 607BD0E8
+U 1 1 60A41526
 P 4950 2000
-AR Path="/607BD0E8" Ref="#PWR?"  Part="1"
-AR Path="/607B2C9D/607BD0E8" Ref="#PWR?"  Part="1"
+AR Path="/60A41526" Ref="#PWR?"  Part="1"
+AR Path="/607B2C9D/60A41526" Ref="#PWR?"  Part="1"
+AR Path="/60A3FFA8/60A41526" Ref="#PWR?"  Part="1"
 F 0 "#PWR?" H 4950 1850 50  0001 C CNN
 F 1 "+5V" H 4965 2173 50  0000 C CNN
