File: .kicad_proj/222.sch (KiCad schematic (older format))
At the start: 6 parts, among them SW1 SW_Push, U1 ATmega328-PU, U2 ADG417BN

Commit message: Finish 2.2.3, change R values in 2.2.7, change 3-state switch component in 2.2.2
Parts:
- removed U2: ADG417BN, Package_DIP:DIP-8_W7.62mm, symbol Analog_Switch:ADG417BN
- added SW2: SW_SPDT, symbol Switch:SW_SPDT
Connections:
- wire segments 16 -> 15
Changed lines of the file:
@@
-$EndComp
-$Comp
-L Analog_Switch:ADG417BN U?
-U 1 1 607C973A
-P 6275 3900
-AR Path="/607C973A" Ref="U?"  Part="1"
-AR Path="/607B2947/607C973A" Ref="U2"  Part="1"
-F 0 "U2" H 6275 4167 50  0000 C CNN
-F 1 "ADG417BN" H 6275 4076 50  0000 C CNN
-F 2 "Package_DIP:DIP-8_W7.62mm" H 6275 3800 50  0001 C CNN
-F 3 "https://www.analog.com/media/en/technical-documentation/data-sheets/ADG417.pdf" H 6275 3900 50  0001 C CNN
-	1    6275 3900
-	1    0    0    -1
 $EndComp
 $Comp
 L power:GND #PWR?
 U 1 1 607C9740
-P 6575 4075
+P 6675 4375
 AR Path="/607C9740" Ref="#PWR?"  Part="1"
 AR Path="/607B2947/607C9740" Ref="#PWR?"  Part="1"
-F 0 "#PWR?" H 6575 3825 50  0001 C CNN
-F 1 "GND" H 6580 3902 50  0000 C CNN
-F 2 "" H 6575 4075 50  0001 C CNN
-F 3 "" H 6575 4075 50  0001 C CNN
-	1    6575 4075
+F 0 "#PWR?" H 6675 4125 50  0001 C CNN
+F 1 "GND" H 6680 4202 50  0000 C CNN
+F 2 "" H 6675 4375 50  0001 C CNN
+F 3 "" H 6675 4375 50  0001 C CNN
+	1    6675 4375
 	1    0    0    -1
 $EndComp
 Wire Wire Line
-	6575 3900 6575 4075
+	6675 4200 6675 4375
 Wire Wire Line
 	5425 4100 5425 2950
@@
 L power:+5V #PWR?
 U 1 1 607C974A
-P 5950 3700
+P 6675 3800
 AR Path="/607C974A" Ref="#PWR?"  Part="1"
 AR Path="/607B2947/607C974A" Ref="#PWR?"  Part="1"
-F 0 "#PWR?" H 5950 3550 50  0001 C CNN
-F 1 "+5V" H 5965 3873 50  0000 C CNN
-F 2 "" H 5950 3700 50  0001 C CNN
-F 3 "" H 5950 3700 50  0001 C CNN
-	1    5950 3700
+F 0 "#PWR?" H 6675 3650 50  0001 C CNN
+F 1 "+5V" H 6690 3973 50  0000 C CNN
+F 2 "" H 6675 3800 50  0001 C CNN
+F 3 "" H 6675 3800 50  0001 C CNN
+	1    6675 3800
 	1    0    0    -1
 $EndComp
 Wire Wire Line
-	5950 3700 5950 3900
-Wire Wire Line
-	5950 3900 5975 3900
+	6675 3800 6675 4000
 $Comp
 L Device:R R?
@@
 	0    1    1    0
 $EndComp
+$Comp
+L Switch:SW_SPDT SW2
+U 1 1 60A12169
+P 6475 4100
+F 0 "SW2" H 6475 4385 50  0000 C CNN
+F 1 "SW_SPDT" H 6475 4294 50  0000 C CNN
+F 2 "" H 6475 4100 50  0001 C CNN
+F 3 "~" H 6475 4100 50  0001 C CNN
+	1    6475 4100
+	1    0    0    -1
+$EndComp
 $EndSCHEMATC
