File: .kicad_proj/226.sch (KiCad schematic (older format))
At the start: 3 parts, among them U1 ATmega328-PU

Commit message: Finish 2.2.3, change R values in 2.2.7, change 3-state switch component in 2.2.2
Connections:
- net +5V: now also U1.20 (AVCC)
Changed lines of the file:
@@
 Wire Wire Line
 	6425 3925 6425 4100
+Wire Wire Line
+	4950 2725 4850 2725
+Connection ~ 4850 2725
 $EndSCHEMATC
