File: .kicad_proj/kicad_proj.sch (KiCad schematic (older format))
At the start: 0 parts

Commit message: Add schematics 9, 10, 11 and 12
Changed lines of the file:
@@
 $Descr A4 11693 8268
 encoding utf-8
-Sheet 1 9
+Sheet 1 19
 Title ""
 Date ""
@@
 F1 "228.sch" 50
 $EndSheet
+$Sheet
+S 2250 1475 500  150
+U 60A4150D
+F0 "sheet2310" 50
+F1 "2310.sch" 50
+$EndSheet
+$Sheet
+S 2250 1100 500  150
+U 60A3FFA8
+F0 "sheet239" 50
+F1 "239.sch" 50
+$EndSheet
+$Sheet
+S 2250 1900 500  150
+U 60A41579
+F0 "sheet2311" 50
+F1 "2311.sch" 50
+$EndSheet
+$Sheet
+S 2250 2300 500  150
+U 60A415AD
+F0 "sheet2312" 50
+F1 "2312.sch" 50
+$EndSheet
+$Sheet
+S 2250 2675 500  150
+U 60A415EB
+F0 "sheet2313" 50
+F1 "2313.sch" 50
+$EndSheet
+$Sheet
+S 3225 1100 500  150
+U 60A41615
+F0 "sheet60A41613" 50
+F1 "2414.sch" 50
+$EndSheet
+$Sheet
+S 3225 1475 500  150
+U 60A41656
+F0 "sheet2315" 50
+F1 "2315.sch" 50
+$EndSheet
+$Sheet
+S 3200 1900 500  150
+U 60A41762
+F0 "sheet2316" 50
+F1 "2316.sch" 50
+$EndSheet
+$Sheet
+S 3200 2300 500  150
+U 60A41786
+F0 "sheet2317" 50
+F1 "2317.sch" 50
+$EndSheet
+$Sheet
+S 3200 2675 500  150
+U 60A417A5
+F0 "sheet2318" 50
+F1 "2318.sch" 50
+$EndSheet
 $EndSCHEMATC

Commit message: Finish schematics 14-16
Changed lines of the file:
@@
 S 3225 1100 500  150
 U 60A41615
-F0 "sheet60A41613" 50
+F0 "sheet14" 50
 F1 "2414.sch" 50
 $EndSheet
