File: .kicad_proj/2318.sch (KiCad schematic (older format))
At the start: 1 part, among them U1 ATmega328-PU

Commit message: Add schematics 18
Parts:
- added J1: Micro_SD_Card, symbol Connector:Micro_SD_Card
Connections:
- net GND: now also J1.6 (VSS)
- net at U1.16 (PB2): now also J1.2 (DAT3/CD)
- net at U1.17 (PB3): now also J1.3 (CMD)
- net at U1.18 (PB4): now also J1.7 (DAT0)
- net at U1.19 (PB5): now also J1.5 (CLK)
- net +5V renamed +3V3
- net +3V3: now also J1.4 (VDD)
Other:
- note added: "CLK"
- note added: "CS"
- note added: "MISO"
- note added: "MOSI"
Changed lines of the file:
@@
 $Descr A4 11693 8268
 encoding utf-8
-Sheet 10 19
+Sheet 19 19
 Title ""
 Date ""
@@
 AR Path="/60A41762/60A41830" Ref="U?"  Part="1"
 AR Path="/60A41786/60A41830" Ref="U?"  Part="1"
-AR Path="/60A417A5/60A41830" Ref="U?"  Part="1"
+AR Path="/60A417A5/60A41830" Ref="U1"  Part="1"
 AR Path="/60A417E2/60A41830" Ref="U?"  Part="1"
-F 0 "U?" H 4306 3546 50  0000 R CNN
+F 0 "U1" H 4306 3546 50  0000 R CNN
 F 1 "ATmega328-PU" H 4306 3455 50  0000 R CNN
 F 2 "Package_DIP:DIP-28_W7.62mm" H 4950 3500 50  0001 C CIN
@@
 L power:GND #PWR?
 U 1 1 60A4182E
-P 4950 5000
+P 4950 5075
 AR Path="/60A4182E" Ref="#PWR?"  Part="1"
 AR Path="/607B2C9D/60A4182E" Ref="#PWR?"  Part="1"
@@
 AR Path="/60A417A5/60A4182E" Ref="#PWR?"  Part="1"
 AR Path="/60A417E2/60A4182E" Ref="#PWR?"  Part="1"
-F 0 "#PWR?" H 4950 4750 50  0001 C CNN
-F 1 "GND" H 4955 4827 50  0000 C CNN
-F 2 "" H 4950 5000 50  0001 C CNN
-F 3 "" H 4950 5000 50  0001 C CNN
-	1    4950 5000
+F 0 "#PWR?" H 4950 4825 50  0001 C CNN
+F 1 "GND" H 4955 4902 50  0000 C CNN
+F 2 "" H 4950 5075 50  0001 C CNN
+F 3 "" H 4950 5075 50  0001 C CNN
+	1    4950 5075
 	1    0    0    -1
 $EndComp
 $Comp
-L power:+5V #PWR?
-U 1 1 60A4182F
-P 4950 2000
-AR Path="/60A4182F" Ref="#PWR?"  Part="1"
-AR Path="/607B2C9D/60A4182F" Ref="#PWR?"  Part="1"
-AR Path="/60A3FFA8/60A4182F" Ref="#PWR?"  Part="1"
-AR Path="/60A4150D/60A4182F" Ref="#PWR?"  Part="1"
-AR Path="/60A41656/60A4182F" Ref="#PWR?"  Part="1"
-AR Path="/60A41762/60A4182F" Ref="#PWR?"  Part="1"
-AR Path="/60A41786/60A4182F" Ref="#PWR?"  Part="1"
-AR Path="/60A417A5/60A4182F" Ref="#PWR?"  Part="1"
-AR Path="/60A417E2/60A4182F" Ref="#PWR?"  Part="1"
-F 0 "#PWR?" H 4950 1850 50  0001 C CNN
-F 1 "+5V" H 4965 2173 50  0000 C CNN
-F 2 "" H 4950 2000 50  0001 C CNN
-F 3 "" H 4950 2000 50  0001 C CNN
-	1    4950 2000
+L Connector:Micro_SD_Card J1
+U 1 1 60B5283B
+P 7675 3425
+F 0 "J1" H 7625 4142 50  0000 C CNN
+F 1 "Micro_SD_Card" H 7625 4051 50  0000 C CNN
+F 2 "" H 8825 3725 50  0001 C CNN
+F 3 "http://katalog.we-online.de/em/datasheet/693072010801.pdf" H 7675 3425 50  0001 C CNN
+	1    7675 3425
 	1    0    0    -1
 $EndComp
+Wire Wire Line
+	6775 3525 5750 3525
+Wire Wire Line
+	5750 3525 5750 2800
+Wire Wire Line
+	5750 2800 5550 2800
+$Comp
+L power:+3.3V #PWR?
+U 1 1 60B58344
+P 4950 1875
+F 0 "#PWR?" H 4950 1725 50  0001 C CNN
+F 1 "+3.3V" H 4965 2048 50  0000 C CNN
+F 2 "" H 4950 1875 50  0001 C CNN
+F 3 "" H 4950 1875 50  0001 C CNN
+	1    4950 1875
+	1    0    0    -1
+$EndComp
+Wire Wire Line
+	6775 3225 5900 3225
+Wire Wire Line
+	5900 3225 5900 2500
+Wire Wire Line
+	5900 2500 5550 2500
+Text Notes 5600 2500 0    50   ~ 0
+CS
+Text Notes 5600 2800 0    50   ~ 0
+CLK
+Wire Wire Line
+	6775 3425 6525 3425
+Wire Wire Line
+	6525 3425 6525 1925
+Wire Wire Line
+	4950 1875 4950 1925
+Connection ~ 4950 1925
+Wire Wire Line
+	4950 1925 4950 2000
+Wire Wire Line
+	4950 5075 4950 5025
+Wire Wire Line
+	4950 5025 6675 5025
+Wire Wire Line
+	6675 5025 6675 3625
+Wire Wire Line
+	6675 3625 6775 3625
+Connection ~ 4950 5025
+Wire Wire Line
+	4950 5025 4950 5000
+Text Notes 5600 2600 0    50   ~ 0
+MOSI
+Text Notes 5600 2700 0    50   ~ 0
+MISO
+Wire Wire Line
+	5550 2600 5875 2600
+Wire Wire Line
+	5875 2600 5875 3325
+Wire Wire Line
+	5875 3325 6775 3325
+Wire Wire Line
+	6775 3725 5800 3725
+Wire Wire Line
+	5800 3725 5800 2700
+Wire Wire Line
+	5800 2700 5550 2700
+Wire Wire Line
+	4950 1925 6525 1925
 $EndSCHEMATC
