File: .kicad_proj/225.sch (KiCad schematic (older format))
At the start: 2 parts, among them U1 ATmega328-PU

Commit message: Finish 2.2.3, change R values in 2.2.7, change 3-state switch component in 2.2.2
Connections:
- net +5V: now also U1.20 (AVCC)
Changed lines of the file:
@@
 	5900 2075 4975 2075
 Connection ~ 4975 2075
-Wire Wire Line
-	4975 2075 4975 2225
 $Comp
 L power:GND #PWR?
@@
 Wire Wire Line
 	6050 3425 5575 3425
+Wire Wire Line
+	4975 2075 4975 2225
+Wire Wire Line
+	5075 2225 4975 2225
+Connection ~ 4975 2225
 $EndSCHEMATC

Commit message: Add resistors
Parts:
- added R1: 100R, symbol Device:R
Connections:
- net at U1.23 (PC0): now also R1.2; no longer RV1.2
- new net: R1.1, RV1.2
Changed lines of the file:
@@
 	6375 2075 6375 2125
-Wire Wire Line
-	6050 2225 6050 3425
 Wire Wire Line
 	6050 3425 5575 3425
@@
 	5075 2225 4975 2225
 Connection ~ 4975 2225
+$Comp
+L Device:R R1
+U 1 1 60D4CC34
+P 6050 3050
+F 0 "R1" H 6120 3096 50  0000 L CNN
+F 1 "100R" H 6120 3005 50  0000 L CNN
+F 2 "" V 5980 3050 50  0001 C CNN
+F 3 "~" H 6050 3050 50  0001 C CNN
+	1    6050 3050
+	1    0    0    -1
+$EndComp
+Wire Wire Line
+	6050 3200 6050 3425
+Wire Wire Line
+	6050 2225 6050 2900
 $EndSCHEMATC
