File: .kicad_proj/2317.sch (KiCad schematic (older format))
At the start: 1 part, among them U1 ATmega328-PU

Commit message: Add schematic 17
Parts:
- added C1, C10, C2, C3, C4, C5, C6, C7, C8, C9: 0.1uF, symbol Device:CP
- added J1, J2: DB9_Female, symbol Connector:DB9_Female
- added U1: ATmega328-PU, Package_DIP:DIP-28_W7.62mm, symbol MCU_Microchip_ATmega:ATmega328-PU
- added U3, U4: MAX232, symbol Interface_UART:MAX232
Connections:
- net +5V: now also C10.1, C4.2, C5.2, C9.1, U1.7 (VCC), U3.16 (VCC), U4.16 (VCC)
- net GND: now also C10.2, C3.1, C8.2, C9.2, J1.5, U1.22 (GND), U1.8 (GND), U3.15 (GND), U4.15 (GND)
- net at U1.2 (PD0): now also U4.12 (R1OUT)
- net at U1.3 (PD1): now also U4.11 (T1IN)
- new net: C1.1, U3.1 (C1+)
- new net: U1.3 (PD1), U3.11 (T1IN)
- new net: U1.2 (PD0), U3.12 (R1OUT)
- new net: J1.3, U3.13 (R1IN)
- new net: J1.2, U3.14 (T1OUT)
- new net: C4.1, U3.2 (VS+)
- new net: C1.2, U3.3 (C1-)
- new net: C2.1, U3.4 (C2+)
- new net: C2.2, U3.5 (C2-)
- new net: C3.2, U3.6 (VS-)
- new net: C6.1, U4.1 (C1+)
- new net: J2.3, U4.13 (R1IN)
- new net: J2.2, U4.14 (T1OUT)
- new net: C5.1, U4.2 (VS+)
- new net: C6.2, U4.3 (C1-)
- new net: C7.1, U4.4 (C2+)
- new net: C7.2, U4.5 (C2-)
- new net: C8.1, U4.6 (VS-)
Other:
- moved on the sheet: U2

Commit message: Add resistors
Parts:
- added R1, R2: 100R, symbol Device:R
Connections:
- net at U1.2 (PD0): now also R2.2; no longer U4.12 (R1OUT)
- net at U3.12 (R1OUT): now also R1.1; no longer U1.2 (PD0)
- new net: R1.2, U1.2 (PD0)
- new net: R2.1, U4.12 (R1OUT)
Changed lines of the file:
@@
 Wire Wire Line
 	2875 4100 2875 4125
-Wire Wire Line
-	2875 4125 2375 4125
 $Comp
 L power:GND #PWR?
@@
 	9325 2950 9250 2950
 Wire Wire Line
-	9250 2950 9250 2550
-Wire Wire Line
-	9250 2550 9025 2550
+	9250 2950 9250 2875
 Wire Wire Line
 	9025 2950 9150 2950
@@
 	1    0    0    -1
 $EndComp
+$Comp
+L Device:R R1
+U 1 1 60D4F920
+P 2600 4125
+F 0 "R1" V 2393 4125 50  0000 C CNN
+F 1 "100R" V 2484 4125 50  0000 C CNN
+F 2 "" V 2530 4125 50  0001 C CNN
+F 3 "~" H 2600 4125 50  0001 C CNN
+	1    2600 4125
+	0    1    1    0
+$EndComp
+$Comp
+L Device:R R2
+U 1 1 60D50D0E
+P 9075 2725
+F 0 "R2" H 9145 2771 50  0000 L CNN
+F 1 "100R" H 9145 2680 50  0000 L CNN
+F 2 "" V 9005 2725 50  0001 C CNN
+F 3 "~" H 9075 2725 50  0001 C CNN
+	1    9075 2725
+	1    0    0    -1
+$EndComp
+Wire Wire Line
+	2450 4125 2375 4125
+Wire Wire Line
+	2750 4125 2875 4125
+Wire Wire Line
+	9075 2575 9075 2550
+Wire Wire Line
+	9075 2550 9025 2550
+Wire Wire Line
+	9075 2875 9250 2875
 $EndSCHEMATC
