File: .kicad_proj/2310.sch (KiCad schematic (older format))
At the start: 17 parts, among them M1 Motor_Servo, M2 Motor_Servo, M3 Motor_Servo, M4 Motor_Servo, M5 Motor_Servo, M6 Motor_Servo, U1 ATmega328-PU, U2 MC7905

Commit message: Fix schematics 10
Parts:
- added C10, C12, C14: 1uF, symbol Device:CP1_Small
- added C11, C13, C9: 0.33uF, symbol Device:CP1_Small
- added U3, U4, U5: MC7905, symbol Regulator_Linear:MC7905
Connections:
- net at BT1.2 (-), C1.2, C2.2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: now also C10.2, C11.2, C12.2, C13.2, C14.2, C9.2, U3.1 (GND), U4.1 (GND), U5.1 (GND)
- net at C7.1, U2.3 (VO): now also U1.7 (VCC); no longer BT1.1 (+)
- new net: BT1.1 (+), C10.1, C12.1, C14.1, C8.1, U2.2 (VI), U3.2 (VI), U4.2 (VI), U5.2 (VI)
- new net: C13.1, C5.1, C6.1, M5.2 (+), M6.2 (+), U5.3 (VO)
- new net: C11.1, C3.1, C4.1, M3.2 (+), M4.2 (+), U4.3 (VO)
- new net: C1.1, C2.1, C9.1, M1.2 (+), M2.2 (+), U3.3 (VO)
Other:
- moved on the sheet: BT1, C7, C8, U2
